File: hardware/Bugcon_2024_Community/Bugcon_2024_Community.kicad_pcb (KiCad board)
At the start: 2 copper layers, 99.7 x 86.6 mm, 55 parts, among them J2 Add_On, J3 OLED, J4 Battery, J5 Battery, P1 USB_C_Plug_USB2.0, Q1 DMG3415U-7, SW1 ON, U1 ESP32-C6-WROOM-1U-N4, U2 XC6220B331MR-G

Commit message: feat: add more labels
Parts:
- added kibuzzard-66FD9F77: G***, kibuzzard-66FD9F77, B.Cu at (85.0, 98.4)
- moved G*** 7.32 mm to (127.0, 71.7)
Other:
- board text added: "Este es el final del camino gracias por acompañarnos LATAM El luchador, el dragon, la llama y BugCon te dan las gracias - Dijo el Gato"
- board text added: "https://github.com/ElectronicCats/badge-bugcon-2024"

Commit message: feat(Hw):Update_Labels_And_route
Parts:
- added kibuzzard-6700283A: G***, kibuzzard-6700283A, B.Cu at (156.0, 117.9)
Changed lines of the file:
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@@
 		)
 	)
+	(footprint "kibuzzard-6700283A"
+		(layer "B.Cu")
+		(at 156.02 117.9 180)
+		(descr "Generated with KiBuzzard")
+		(tags "kb_params=eyJBbGlnbm1lbnRDaG9pY2UiOiAiQ2VudGVyIiwgIkNhcExlZnRDaG9pY2UiOiAiWyIsICJDYXBSaWdodENob2ljZSI6ICJdIiwgIkZvbnRDb21ib0JveCI6ICJVYnVudHVNb25vLUIiLCAiSGVpZ2h0Q3RybCI6IDEuMCwgIkxheWVyQ29tYm9Cb3giOiAiRi5TaWxrUyIsICJMaW5lU3BhY2luZ0N0cmwiOiAxLjUsICJNdWx0aUxpbmVUZXh0IjogInYxLjFcclxuIiwgIlBhZGRpbmdCb3R0b21DdHJsIjogMS4wLCAiUGFkZGluZ0xlZnRDdHJsIjogMi41LCAiUGFkZGluZ1JpZ2h0Q3RybCI6IDIuNSwgIlBhZGRpbmdUb3BDdHJsIjogMS4wLCAiV2lkdGhDdHJsIjogMS4wfQ==")
+		(property "Reference" "kibuzzard-6700283A"
+			(at 0 3.680275 0)
+			(layer "B.SilkS")
+			(hide yes)
+			(effects
+				(font
+					(size 0.001 0.001)
+				)
+				(justify mirror)
+			)
+		)
+		(property "Value" "G***"
+			(at 0 -3.680275 0)
+			(layer "B.SilkS")
+			(hide yes)
+			(effects
+				(font
+					(size 0.001 0.001)
+				)
+				(justify mirror)
+			)
+		)
+		(property "Footprint" ""
+			(at 0 0 0)
+			(layer "B.Fab")
+			(hide yes)
+			(effects
+				(font
+					(size 1.27 1.27)
+					(thickness 0.15)
+				)
+				(justify mirror)
+			)
+		)
+		(property "Datasheet" ""
+			(at 0 0 0)
+			(layer "B.Fab")
+			(hide yes)
+			(effects
+				(font
+					(size 1.27 1.27)
+					(thickness 0.15)
+				)
+				(justify mirror)
+			)
+		)
+		(property "Description" ""
+			(at 0 0 0)
+			(layer "B.Fab")
+			(hide yes)
+			(effects
+				(font
+					(size 1.27 1.27)
+					(thickness 0.15)
+				)
+				(justify mirror)
+			)
+		)
+		(attr board_only exclude_from_pos_files exclude_from_bom)
+		(fp_poly
+			(pts
+				(xy -1.543651 0.632275) (xy -1.874339 0.632275) (xy -1.874339 -0.632275) (xy -1.543651 -0.632275)
+				(xy -1.257937 -0.632275) (xy -1.257937 -0.48254) (xy -1.30582 -0.382981) (xy -1.354233 -0.272663)
+				(xy -1.403175 -0.151587) (xy -1.439633 -0.054514) (xy -1.475198 0.047024) (xy -1.509871 0.153026)
+				(xy -1.543651 0.263492) (xy -1.338889 0.263492) (xy -1.323214 0.20119) (xy -1.304762 0.134921) (xy -1.284325 0.066468)
+				(xy -1.262698 -0.002381) (xy -1.240278 -0.070437) (xy -1.21746 -0.136508) (xy -1.17381 -0.255556)
+				(xy -1.127778 -0.136508) (xy -1.102579 -0.070437) (xy -1.077778 -0.002381) (xy -1.053571 0.066468)
+				(xy -1.030159 0.134921) (xy -1.009325 0.20119) (xy -0.992857 0.263492) (xy -0.794444 0.263492) (xy -0.828671 0.153026)
+				(xy -0.864683 0.047024) (xy -0.90248 -0.054514) (xy -0.942063 -0.151587) (xy -0.994974 -0.272663)
+				(xy -1.045767 -0.382981) (xy -1.094444 -0.48254) (xy -1.257937 -0.48254) (xy -1.257937 -0.632275)
+				(xy -0.043651 -0.632275) (xy -0.043651 -0.48254) (xy -0.640476 -0.48254) (xy -0.640476 -0.320635)
+				(xy -0.434127 -0.320635) (xy -0.434127 0.228571) (xy -0.535714 0.172222) (xy -0.63254 0.133333)
+				(xy -0.696032 0.295238) (xy -0.613492 0.331746) (xy -0.524603 0.380952) (xy -0.440476 0.438095)
+				(xy -0.372222 0.5) (xy -0.238889 0.5) (xy -0.238889 -0.320635) (xy -0.043651 -0.320635) (xy -0.043651 -0.48254)
+				(xy -0.043651 -0.632275) (xy 0.419841 -0.632275) (xy 0.419841 -0.5) (xy 0.365873 -0.490476) (xy 0.320635 -0.462698)
+				(xy 0.288889 -0.418254) (xy 0.276984 -0.357143) (xy 0.288889 -0.297619) (xy 0.320635 -0.253968)
+				(xy 0.365873 -0.226984) (xy 0.419841 -0.21746) (xy 0.518254 -0.253968) (xy 0.561111 -0.357143) (xy 0.518254 -0.463492)
+				(xy 0.419841 -0.5) (xy 0.419841 -0.632275) (xy 1.543651 -0.632275) (xy 1.543651 -0.48254) (xy 0.946825 -0.48254)
+				(xy 0.946825 -0.320635) (xy 1.153175 -0.320635) (xy 1.153175 0.228571) (xy 1.051587 0.172222) (xy 0.954762 0.133333)
+				(xy 0.89127 0.295238) (xy 0.97381 0.331746) (xy 1.062698 0.380952) (xy 1.146825 0.438095) (xy 1.215079 0.5)
+				(xy 1.348413 0.5) (xy 1.348413 -0.320635) (xy 1.543651 -0.320635) (xy 1.543651 -0.48254) (xy 1.543651 -0.632275)
+				(xy 1.874339 -0.632275) (xy 1.874339 0.632275) (xy 1.543651 0.632275) (xy -1.543651 0.632275)
+			)
+			(stroke
+				(width 0)
+				(type solid)
+			)
+			(fill solid)
+			(layer "B.SilkS")
+		)
+	)
 	(footprint "Capacitor_SMD:C_0603_1608Metric"
 		(layer "B.Cu")
@@
 	)
 	(gr_text "https://github.com/ElectronicCats/badge-bugcon-2024"
-		(at 150.51 86.62 0)
+		(at 149.05 86.57 0)
 		(layer "B.SilkS")
 		(effects
@@
 	)
 	(segment
-		(start 155.120515 117.750515)
-		(end 158.243802 117.750515)
-		(width 0.4)
-		(layer "F.Cu")
-		(net 2)
-	)
-	(segment
 		(start 105.65 90.26)
 		(end 105.64 90.25)
@@
 	)
 	(segment
-		(start 151.943802 117.750515)
-		(end 155.119485 117.750515)
-		(width 0.4)
-		(layer "F.Cu")
-		(net 2)
-	)
-	(segment
 		(start 138.105 71.635)
 		(end 137.5 72.24)
@@
 	)
 	(segment
-		(start 155.12 117.75)
-		(end 155.120515 117.750515)
-		(width 0.4)
-		(layer "F.Cu")
-		(net 2)
-	)
-	(segment
 		(start 163.7 104.18)
 		(end 161.23 104.18)
@@
 	)
 	(segment
+		(start 153.63 117.750515)
+		(end 158.243802 117.750515)
+		(width 0.4)
+		(layer "F.Cu")
+		(net 2)
+	)
+	(segment
 		(start 89.199485 111.920515)
 		(end 89.06 112.06)
@@
 	)
 	(segment
+		(start 153.63 117.750515)
+		(end 151.943802 117.750515)
+		(width 0.4)
+		(layer "F.Cu")
+		(net 2)
+	)
+	(segment
 		(start 80.249485 110.120515)
 		(end 80.27 110.1)
@@
 	)
 	(segment
-		(start 155.119485 117.750515)
-		(end 155.12 117.75)
-		(width 0.4)
-		(layer "F.Cu")
-		(net 2)
-	)
-	(segment
 		(start 137.87 73.96)
 		(end 137.85 73.94)
@@
 	)
 	(via
-		(at 155.12 117.75)
+		(at 153.63 117.750515)
 		(size 0.6)
 		(drill 0.3)
